Commit message: fixing the URDF to have the correct front/back, updating the IMU location

File: segway_v3/segway_description/urdf/segway_components/segway_base.urdf.xacro (robot description, xacro)
@@ -64,46 +64,4 @@
             <child link="base_chassis_link" />
         </joint>
-        <!-- Front caster -->
-        <link name="front_caster_wheel_link">
-			<collision>
-			    <origin xyz="0 0 0" rpy="0 0 0"/>
-				<geometry>
-				    <sphere radius="0.083567"/>
-				</geometry>
-			</collision>
-		</link>
-        <joint name="front_caster_wheel_joint" type="fixed">
-            <origin xyz="0.370050 0 -0.074451" rpy="0 0 0" />
-            <parent link="base_chassis_link" />
-            <child link="front_caster_wheel_link" />
-        </joint>
-		<gazebo reference="front_caster_wheel_link">
-            <kp>1000000.0</kp>
-            <kd>10.0</kd>
-            <mu1>0</mu1>
-            <mu2>0</mu2>
-            <minDepth>0.003</minDepth>
-        </gazebo>
-        <!-- Rear caster -->
-        <link name="rear_caster_wheel_link">
-			<collision>
-			    <origin xyz="0 0 0" rpy="0 0 0"/>
-				<geometry>
-				    <sphere radius="0.083567"/>
-				</geometry>
-			</collision>
-		</link>
-        <joint name="rear_caster_wheel_joint" type="fixed">
-            <origin xyz="-0.370050 0 -0.074451" rpy="0 0 0" />
-            <parent link="base_chassis_link" />
-            <child link="rear_caster_wheel_link" />
-        </joint>
-		<gazebo reference="rear_caster_wheel_link">
-            <kp>1000000.0</kp>
-            <kd>10.0</kd>
-            <mu1>0</mu1>
-            <mu2>0</mu2>
-            <minDepth>0.003</minDepth>
-        </gazebo>
         <!-- Segway wheel macros -->
         <xacro:i2_wheel wheel_prefix="left" parent="base_chassis_link" visual_rotation="0.0">

File: segway_v3/segway_description/urdf/sensors/segway_sensors.urdf.xacro (robot description, xacro)
@@ -27,5 +27,5 @@
         <link name="imu_frame"/>
         <joint name="imu_joint" type="fixed">
-            <origin xyz="-0.064612 -0.117995 0.08078" rpy="0 0 0" />
+            <origin xyz="-0.063902 -0.095661 0.094815" rpy="0 0 0" />
             <parent link="base_chassis_link" />
             <child link="imu_frame" />
